File: pcbs/KLON (11).kicad_pcb (KiCad board)
At the start: 2 copper layers, 159.6 x 117.7 mm, 91 parts, among them J1 MJ-4PP-9, SW25 Rotary_Encoder_Switch

Commit message: updateed jumper and added that to pcb
Connections:
- SSD1306 pad 3: SCL -> jump
Routing:
- net GND: track 29.5 -> 143.6 mm, vias 0 -> 1
- net RST: track 9.84 -> 78.2 mm
- net P9: track 9.83 -> 73.8 mm
- net BAT_P: track 0.00 -> 49.2 mm
- net VCC: track 9.84 -> 57.9 mm
- net P16: track 38.5 -> 64.1 mm
- net P10: track 38.5 -> 58.5 mm
- net 4_r0: track 32.3 -> 51.7 mm
- net RAW: track 9.84 -> 27.7 mm, vias 0 -> 1
- net jump: track 0.00 -> 9.08 mm
- net RX: track 0.00 -> 5.95 mm
- net TX: track 0.00 -> 2.45 mm
- net 2_r0: track 32.3 -> 34.7 mm
- net 3_r0: track 32.3 -> 34.7 mm
- net 1_r0: track 32.3 -> 34.6 mm
