File: pcbs/KLON -nice_view.kicad_pcb (KiCad board)
At the start: 2 copper layers, 159.6 x 117.7 mm, 88 parts, among them J1 MJ-4PP-9, SW25 Rotary_Encoder_Switch

Commit message: added some pcb stuff
Parts:
- moved RST1 3.22 mm to (134.0, 161.6)
- moved D18 3.22 mm to (194.7, 178.1)
- moved S19 3.22 mm to (173.6, 172.5)
- moved S40 3.22 mm to (173.6, 172.5)
- moved D7 3.22 mm to (210.8, 147.1)
- moved D1 3.22 mm to (172.8, 160.1)
- moved S26 3.22 mm to (191.8, 128.6)
- moved S5 3.22 mm to (191.8, 128.6)
- moved S29 3.22 mm to (210.8, 119.6)
- moved S8 3.22 mm to (210.8, 119.6)
- moved XX7 3.22 mm to (151.9, 143.8)
- moved D13 3.22 mm to (246.2, 171.4)
- moved SW25 3.22 mm to (147.3, 155.8)
- moved MH6 3.22 mm to (230.8, 163.5)
- moved D4 3.22 mm to (191.8, 156.1)
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Connections:
- D22 pad 1: P2 -> SW18B
- D22 pad 2: P2 -> SW18B
- SSD1306 pad 1: GND -> dis1-pad4
- SSD1306 pad 2: VCC -> dis1-pad3
- SSD1306 pad 3: SCL -> dis1-pad2
- SSD1306 pad 4: SDA -> dis1-pad1
- SW25 pad MP: undefined -> (no net)
- SW25 pad S1: col -> P3
- SW25 pad S2: row -> SW18B
- XX4 pad 1: P2 -> dis1-pad1
- XX4 pad 2: P1 -> GND
- XX5 pad 1: P2 -> dis1-pad2
- XX5 pad 2: P1 -> VCC
- XX6 pad 1: P2 -> dis1-pad3
- XX6 pad 2: P1 -> SCL
- XX7 pad 1: P2 -> dis1-pad4
- XX7 pad 2: P1 -> SDA
Routing:
- net row3: track 0.00 -> 145.5 mm
- net row2: track 0.00 -> 125.3 mm
- net P3: track 124.7 -> 243.5 mm
- net P4: track 124.7 -> 229.0 mm
- net row1: track 0.00 -> 100.3 mm
- net VCC: track 9.84 -> 96.7 mm, vias 0 -> 1
- net RST: track 9.84 -> 87.2 mm, vias 0 -> 1
- net P5: track 96.0 -> 172.0 mm
- net P6: track 96.0 -> 170.0 mm
- net row4: track 0.00 -> 62.6 mm
- net P7: track 96.0 -> 157.3 mm, vias 6 -> 8
- net BAT_P: track 0.00 -> 46.0 mm, vias 0 -> 1
- net P8: track 67.2 -> 104.2 mm, vias 4 -> 6
- net pinky_home: track 32.3 -> 64.5 mm
- net pinky_extra_home: track 32.3 -> 64.5 mm
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- added copper zone on B.Cu, net GND
- added copper zone on F.Cu, net GND
Other:
- outline, holes or cut-outs redrawn

Commit message: finished pcb v1
Routing:
- net GND: track 61.6 -> 76.9 mm, vias 10 -> 14
Other:
- board text added: "SSD1306"
