File: pcbs/KLON -nice_view - Copy.kicad_pcb (KiCad board)
At the start: 2 copper layers, 159.6 x 117.7 mm, 88 parts, among them J1 MJ-4PP-9, SW25 Rotary_Encoder_Switch

Commit message: klon pcb v2
Parts:
- moved D9 3.22 mm to (212.0, 112.1)
- moved D19 3.22 mm to (177.1, 183.6)
- moved D3 3.22 mm to (174.0, 125.1)
- moved H2 3.22 mm to (183.5, 140.3)
- moved D11 3.22 mm to (231.8, 141.4)
- moved D18 3.22 mm to (196.0, 181.1)
- moved MH5 3.22 mm to (247.0, 119.9)
- moved MH6 3.22 mm to (232.0, 166.4)
- moved MH9 3.22 mm to (136.3, 180.0)
- moved XX4 3.22 mm to (145.6, 146.7)
- moved DISP1 3.22 mm to (150.0, 120.6)
- moved D5 3.22 mm to (193.0, 140.1)
- moved D8 3.22 mm to (212.0, 131.1)
- moved S24 3.22 mm to (174.0, 116.6)
- moved S3 3.22 mm to (174.0, 116.6)
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Other:
- outline, holes or cut-outs redrawn
- board text added: "K"
- board text added: "KLON"
- board text added: "L"
- board text added: "N"
- board text added: "O"
- board text added: "REVISION 1.4 BY GEIST + THEB0B, and LU"
- board text added: "SSD1306"
