File: pcbs/KLON -nice_view - Copy2.kicad_pcb (KiCad board)
At the start: 2 copper layers, 159.6 x 117.7 mm, 88 parts, among them J1 MJ-4PP-9, SW25 Rotary_Encoder_Switch

Commit message: pcb update
Parts:
- moved MH3 1.28 mm to (227.7, 101.9)
- moved D18 1.28 mm to (196.5, 182.2)
- moved S11 1.28 mm to (232.9, 134.1)
- moved S32 1.28 mm to (232.9, 134.1)
- moved XX4 1.28 mm to (146.1, 147.9)
- moved S17 1.28 mm to (272.3, 146.8)
- moved S27 1.28 mm to (193.6, 113.8)
- moved S29 1.28 mm to (212.6, 123.8)
- moved S38 1.28 mm to (272.3, 146.8)
- moved S6 1.28 mm to (193.6, 113.8)
- moved S8 1.28 mm to (212.6, 123.8)
- moved D17 1.28 mm to (270.9, 155.1)
- moved S16 1.28 mm to (269.0, 165.5)
- moved S37 1.28 mm to (269.0, 165.5)
- moved D1 1.28 mm to (174.6, 164.3)
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Routing:
- net col4: track 390.5 -> 357.6 mm
- net pinky_extra_bottom: track 63.5 -> 50.0 mm
- net pinky_top: track 64.5 -> 53.0 mm
- net pinky_home: track 64.5 -> 54.0 mm
- net pinky_extra_home: track 64.5 -> 54.1 mm
- net row3: track 186.0 -> 191.7 mm
- net col3: track 351.6 -> 356.1 mm
- net col5: track 315.5 -> 319.7 mm
- net RAW: track 26.0 -> 28.9 mm
- net CS: track 42.6 -> 45.4 mm
- net row4: track 139.9 -> 142.3 mm
- net MOSI: track 76.6 -> 79.0 mm
- net BAT_P: track 49.4 -> 51.6 mm
- net col6: track 276.3 -> 277.9 mm
- net RST: track 87.2 -> 85.6 mm
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
Commit message: updated pcb more
Connections:
- MCU1 pad 113: P10 -> TX
- MCU1 pad 114: P16 -> RX
Routing:
- net TX: track 2.45 -> 12.3 mm
- net P10: track 9.84 -> 0.00 mm
- net RX: track 5.95 -> 15.8 mm
- net P16: track 9.84 -> 0.00 mm
Changed lines of the file:
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@@
 			(size 0.2 0.2)
 			(layers "F.Cu" "F.Mask" "F.Paste")
-			(net "P10")
+			(net "TX")
 			(zone_connect 2)
 			(options
@@
 			(layers "*.Cu" "*.Mask")
 			(remove_unused_layers no)
-			(net "P10")
+			(net "TX")
 		)
 		(pad "113" smd custom
@@
 			(size 0.2 0.2)
 			(layers "B.Cu" "B.Mask" "B.Paste")
-			(net "P10")
+			(net "TX")
 			(zone_connect 2)
 			(options
@@
 			(size 0.2 0.2)
 			(layers "F.Cu" "F.Mask" "F.Paste")
-			(net "P16")
+			(net "RX")
 			(zone_connect 2)
 			(options
@@
 			(layers "*.Cu" "*.Mask")
 			(remove_unused_layers no)
-			(net "P16")
+			(net "RX")
 		)
 		(pad "114" smd custom
@@
 			(size 0.2 0.2)
 			(layers "B.Cu" "B.Mask" "B.Paste")
-			(net "P16")
+			(net "RX")
 			(zone_connect 2)
 			(options
@@
 		(fp_line
 			(start -7 -6.2)
-			(end -2.519997 -6.199997)
+			(end -2.519996 -6.199997)
 			(stroke
 				(width 0.15)
@@
 			(start -2.000001 -6.779999)
 			(mid -2.139878 -6.382304)
-			(end -2.519997 -6.199997)
+			(end -2.519996 -6.199997)
 			(stroke
 				(width 0.15)
@@
 		(fp_line
 			(start -7 -6.2)
-			(end -2.519997 -6.199997)
+			(end -2.519996 -6.199997)
 			(stroke
 				(width 0.15)
@@
 			(start -2.000001 -6.779999)
 			(mid -2.139878 -6.382304)
-			(end -2.519997 -6.199997)
+			(end -2.519996 -6.199997)
 			(stroke
 				(width 0.15)
@@
 		(fp_line
 			(start -7 -6.2)
-			(end -2.519997 -6.199997)
+			(end -2.519996 -6.199997)
 			(stroke
 				(width 0.15)
@@
 			(start -2.000001 -6.779999)
 			(mid -2.139878 -6.382304)
-			(end -2.519997 -6.199997)
+			(end -2.519996 -6.199997)
 			(stroke
 				(width 0.15)
@@
 	)
 	(segment
-		(start 145.807306 131.996847)
-		(end 147.182305 131.99685)
-		(width 0.25)
-		(layer "F.Cu")
-		(net "P10")
-	)
-	(segment
-		(start 153.177001 131.776851)
-		(end 147.402308 131.776847)
-		(width 0.25)
-		(layer "B.Cu")
-		(net "P10")
-	)
-	(segment
-		(start 153.681997 131.271848)
-		(end 153.177001 131.776851)
-		(width 0.25)
-		(layer "B.Cu")
-		(net "P10")
-	)
-	(segment
-		(start 155.007611 131.996852)
-		(end 154.282612 131.271851)
-		(width 0.25)
-		(layer "B.Cu")
-		(net "P10")
-	)
-	(segment
-		(start 155.357306 131.996851)
-		(end 155.007611 131.996852)
-		(width 0.25)
-		(layer "B.Cu")
-		(net "P10")
-	)
-	(segment
-		(start 154.282612 131.271851)
-		(end 153.681997 131.271848)
-		(width 0.25)
-		(layer "B.Cu")
-		(net "P10")
-	)
-	(segment
-		(start 145.807311 129.456849)
-		(end 147.18231 129.45685)
-		(width 0.25)
-		(layer "F.Cu")
-		(net "P16")
-	)
-	(segment
-		(start 155.357304 129.456849)
-		(end 155.00761 129.456851)
-		(width 0.25)
-		(layer "B.Cu")
-		(net "P16")
-	)
-	(segment
-		(start 153.682002 128.731851)
-		(end 153.177 129.236852)
-		(width 0.25)
-		(layer "B.Cu")
-		(net "P16")
-	)
-	(segment
-		(start 155.00761 129.456851)
-		(end 154.28261 128.731848)
-		(width 0.25)
-		(layer "B.Cu")
-		(net "P16")
-	)
-	(segment
-		(start 154.28261 128.731848)
-		(end 153.682002 128.731851)
-		(width 0.25)
-		(layer "B.Cu")
-		(net "P16")
-	)
-	(segment
-		(start 153.177 129.236852)
-		(end 147.402306 129.236849)
-		(width 0.25)
-		(layer "B.Cu")
-		(net "P16")
-	)
-	(segment
 		(start 145.807307 126.916848)
 		(end 147.182305 126.916849)
@@
 	)
 	(segment
+		(start 145.807311 129.456849)
+		(end 147.18231 129.45685)
+		(width 0.25)
+		(layer "F.Cu")
+		(net "RX")
+	)
+	(segment
+		(start 155.357304 129.456849)
+		(end 155.00761 129.456851)
+		(width 0.25)
+		(layer "B.Cu")
+		(net "RX")
+	)
+	(segment
+		(start 153.682002 128.731851)
+		(end 153.177 129.236852)
+		(width 0.25)
+		(layer "B.Cu")
+		(net "RX")
+	)
+	(segment
 		(start 137.640306 177.226851)
 		(end 137.640304 171.27685)
@@
 	)
 	(segment
+		(start 155.00761 129.456851)
+		(end 154.28261 128.731848)
+		(width 0.25)
+		(layer "B.Cu")
+		(net "RX")
+	)
+	(segment
+		(start 154.28261 128.731848)
+		(end 153.682002 128.731851)
+		(width 0.25)
+		(layer "B.Cu")
+		(net "RX")
+	)
+	(segment
+		(start 153.177 129.236852)
+		(end 147.402306 129.236849)
+		(width 0.25)
+		(layer "B.Cu")
+		(net "RX")
+	)
+	(segment
+		(start 145.807306 131.996847)
+		(end 147.182305 131.99685)
+		(width 0.25)
+		(layer "F.Cu")
+		(net "TX")
+	)
+	(segment
+		(start 153.177001 131.776851)
+		(end 147.402308 131.776847)
+		(width 0.25)
+		(layer "B.Cu")
+		(net "TX")
+	)
+	(segment
+		(start 153.681997 131.271848)
+		(end 153.177001 131.776851)
+		(width 0.25)
+		(layer "B.Cu")
+		(net "TX")
+	)
+	(segment
+		(start 155.007611 131.996852)
+		(end 154.282612 131.271851)
+		(width 0.25)
+		(layer "B.Cu")
+		(net "TX")
+	)
+	(segment
 		(start 146.140305 175.47685)
 		(end 146.140304 173.02685)
@@
 		(layer "B.Cu")
 		(net "TX")
+	)
+	(segment
+		(start 155.357306 131.996851)
+		(end 155.007611 131.996852)
+		(width 0.25)
+		(layer "B.Cu")
+		(net "TX")
+	)
+	(segment
+		(start 154.282612 131.271851)
+		(end 153.681997 131.271848)
+		(width 0.25)
+		(layer "B.Cu")
+		(net "TX")
